File: Wapuugotchi.brd (EAGLE design)
At the start: 86 x 64.8 mm, 14 parts, among them IC1 MCP170350MB, SW1 BTN B, SW2 BTN C, SW3 BTN A

Commit message: Tweak the hardware to account for how the switch is wired (left side isolated from right)
Connections:
- net N$12: now also S1.3; no longer S1.4
Routing:
- net N$12: track 9.09 -> 13.1 mm, vias 0 -> 2
Changed lines of the file:
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@@
 <signal name="N$12">
 <contactref element="IC1" pad="2@1"/>
-<contactref element="S1" pad="4"/>
-<wire x1="52.07" y1="14.5542" x2="48.5142" y2="18.11" width="0.254" layer="1"/>
-<wire x1="48.5142" y1="18.11" x2="44.45" y2="18.11" width="0.254" layer="1"/>
+<contactref element="S1" pad="3"/>
+<wire x1="52.07" y1="23.5458" x2="52.07" y2="22.86" width="0.254" layer="1"/>
+<wire x1="52.07" y1="22.86" x2="46.99" y2="22.86" width="0.254" layer="1"/>
+<wire x1="44.45" y1="18.11" x2="44.45" y2="22.86" width="0.254" layer="1"/>
+<wire x1="46.99" y1="22.86" x2="44.45" y2="22.86" width="0.254" layer="16"/>
+<via x="44.45" y="22.86" extent="1-16" drill="0.35"/>
+<via x="46.99" y="22.86" extent="1-16" drill="0.35"/>
 </signal>
 </signals>
